File: 60rtho.kicad_sch (KiCad schematic)
At the start: 165 parts, among them SW1 Esc, SW10 9, SW11 0, SW12 -, SW13 =, SW14 Bksp2u, SW15 Bksp1u, SW16 Tab, SW17 Q, SW18 W, SW19 E, SW2 1, SW20 R, SW21 T, SW22 Y, SW23 U, SW24 I, SW25 O, SW26 P, SW27 LBrk, SW28 RBrk, SW29 Bslash, SW3 2, SW30 Bslash15, SW31 Caps, SW32 A, SW33 S, SW34 D, SW35 F, SW36 G, SW37 H, SW38 J, SW39 K, SW4 3, SW40 L, SW41 Semi, SW42 Quote, SW43 Enter, SW44 LShift, SW45 Z, SW46 X, SW47 C, SW48 V, SW49 B, SW5 4, SW50 N, SW51 M, SW52 Comma, SW53 Period, SW54 Slash, SW55 RShift, SW56 Up, SW57 RShift225, SW58 LCtrl, SW59 LWin, SW6 5, SW60 LAlt, SW61 Space625, SW62 Space225, SW63 Space125, SW64 Space275, SW65 RAlt, SW66 RWin, SW67 Menu, SW68 RCtrl, SW69 Left, SW7 6, SW70 Down, SW71 Right, SW8 7, SW9 8

Commit message: Fixed schematic
Parts:
- removed D62, D64, D65, D66, D67, D68, D69, D70, D71: 1N4148W, Diode_SMD:D_SOD-123, symbol Device:D
- removed SW1: Esc, Button_Switch_Keyboard:SW_Cherry_MX_1.00u_PCB, symbol Switch:SW_Push
- removed SW10: 9, Button_Switch_Keyboard:SW_Cherry_MX_1.00u_PCB, symbol Switch:SW_Push
- removed SW11: 0, Button_Switch_Keyboard:SW_Cherry_MX_1.00u_PCB, symbol Switch:SW_Push
- removed SW12: -, Button_Switch_Keyboard:SW_Cherry_MX_1.00u_PCB, symbol Switch:SW_Push
- removed SW13: =, Button_Switch_Keyboard:SW_Cherry_MX_1.00u_PCB, symbol Switch:SW_Push
- removed SW14: Bksp2u, Button_Switch_Keyboard:SW_Cherry_MX_1.00u_PCB, symbol Switch:SW_Push
- removed SW15: Bksp1u, Button_Switch_Keyboard:SW_Cherry_MX_1.00u_PCB, symbol Switch:SW_Push
- removed SW16: Tab, Button_Switch_Keyboard:SW_Cherry_MX_1.00u_PCB, symbol Switch:SW_Push
- removed SW17: Q, Button_Switch_Keyboard:SW_Cherry_MX_1.00u_PCB, symbol Switch:SW_Push
- removed SW18: W, Button_Switch_Keyboard:SW_Cherry_MX_1.00u_PCB, symbol Switch:SW_Push
- removed SW19: E, Button_Switch_Keyboard:SW_Cherry_MX_1.00u_PCB, symbol Switch:SW_Push
- removed SW2: 1, Button_Switch_Keyboard:SW_Cherry_MX_1.00u_PCB, symbol Switch:SW_Push
- removed SW20: R, Button_Switch_Keyboard:SW_Cherry_MX_1.00u_PCB, symbol Switch:SW_Push
- removed SW21: T, Button_Switch_Keyboard:SW_Cherry_MX_1.00u_PCB, symbol Switch:SW_Push
- removed SW22: Y, Button_Switch_Keyboard:SW_Cherry_MX_1.00u_PCB, symbol Switch:SW_Push
- removed SW23: U, Button_Switch_Keyboard:SW_Cherry_MX_1.00u_PCB, symbol Switch:SW_Push
- removed SW24: I, Button_Switch_Keyboard:SW_Cherry_MX_1.00u_PCB, symbol Switch:SW_Push
- removed SW25: O, Button_Switch_Keyboard:SW_Cherry_MX_1.00u_PCB, symbol Switch:SW_Push
- removed SW26: P, Button_Switch_Keyboard:SW_Cherry_MX_1.00u_PCB, symbol Switch:SW_Push
- removed SW27: LBrk, Button_Switch_Keyboard:SW_Cherry_MX_1.00u_PCB, symbol Switch:SW_Push
- removed SW28: RBrk, Button_Switch_Keyboard:SW_Cherry_MX_1.00u_PCB, symbol Switch:SW_Push
- removed SW29: Bslash, Button_Switch_Keyboard:SW_Cherry_MX_1.00u_PCB, symbol Switch:SW_Push
- removed SW3: 2, Button_Switch_Keyboard:SW_Cherry_MX_1.00u_PCB, symbol Switch:SW_Push
- removed SW30: Bslash15, Button_Switch_Keyboard:SW_Cherry_MX_1.00u_PCB, symbol Switch:SW_Push
- removed SW31: Caps, Button_Switch_Keyboard:SW_Cherry_MX_1.00u_PCB, symbol Switch:SW_Push
- removed SW32: A, Button_Switch_Keyboard:SW_Cherry_MX_1.00u_PCB, symbol Switch:SW_Push
- removed SW33: S, Button_Switch_Keyboard:SW_Cherry_MX_1.00u_PCB, symbol Switch:SW_Push
- removed SW34: D, Button_Switch_Keyboard:SW_Cherry_MX_1.00u_PCB, symbol Switch:SW_Push
- removed SW35: F, Button_Switch_Keyboard:SW_Cherry_MX_1.00u_PCB, symbol Switch:SW_Push
- removed SW36: G, Button_Switch_Keyboard:SW_Cherry_MX_1.00u_PCB, symbol Switch:SW_Push
- removed SW37: H, Button_Switch_Keyboard:SW_Cherry_MX_1.00u_PCB, symbol Switch:SW_Push
- removed SW38: J, Button_Switch_Keyboard:SW_Cherry_MX_1.00u_PCB, symbol Switch:SW_Push
- removed SW39: K, Button_Switch_Keyboard:SW_Cherry_MX_1.00u_PCB, symbol Switch:SW_Push
- removed SW4: 3, Button_Switch_Keyboard:SW_Cherry_MX_1.00u_PCB, symbol Switch:SW_Push
- removed SW40: L, Button_Switch_Keyboard:SW_Cherry_MX_1.00u_PCB, symbol Switch:SW_Push
- removed SW41: Semi, Button_Switch_Keyboard:SW_Cherry_MX_1.00u_PCB, symbol Switch:SW_Push
- removed SW42: Quote, Button_Switch_Keyboard:SW_Cherry_MX_1.00u_PCB, symbol Switch:SW_Push
- removed SW43: Enter, Button_Switch_Keyboard:SW_Cherry_MX_1.00u_PCB, symbol Switch:SW_Push
- removed SW44: LShift, Button_Switch_Keyboard:SW_Cherry_MX_1.00u_PCB, symbol Switch:SW_Push
- removed SW45: Z, Button_Switch_Keyboard:SW_Cherry_MX_1.00u_PCB, symbol Switch:SW_Push
- removed SW46: X, Button_Switch_Keyboard:SW_Cherry_MX_1.00u_PCB, symbol Switch:SW_Push
- removed SW47: C, Button_Switch_Keyboard:SW_Cherry_MX_1.00u_PCB, symbol Switch:SW_Push
- removed SW48: V, Button_Switch_Keyboard:SW_Cherry_MX_1.00u_PCB, symbol Switch:SW_Push
- removed SW49: B, Button_Switch_Keyboard:SW_Cherry_MX_1.00u_PCB, symbol Switch:SW_Push
- removed SW5: 4, Button_Switch_Keyboard:SW_Cherry_MX_1.00u_PCB, symbol Switch:SW_Push
- removed SW50: N, Button_Switch_Keyboard:SW_Cherry_MX_1.00u_PCB, symbol Switch:SW_Push
- removed SW51: M, Button_Switch_Keyboard:SW_Cherry_MX_1.00u_PCB, symbol Switch:SW_Push
- removed SW52: Comma, Button_Switch_Keyboard:SW_Cherry_MX_1.00u_PCB, symbol Switch:SW_Push
- removed SW53: Period, Button_Switch_Keyboard:SW_Cherry_MX_1.00u_PCB, symbol Switch:SW_Push
- removed SW54: Slash, Button_Switch_Keyboard:SW_Cherry_MX_1.00u_PCB, symbol Switch:SW_Push
- removed SW55: RShift, Button_Switch_Keyboard:SW_Cherry_MX_1.00u_PCB, symbol Switch:SW_Push
- removed SW56: Up, Button_Switch_Keyboard:SW_Cherry_MX_1.00u_PCB, symbol Switch:SW_Push
- removed SW57: RShift225, Button_Switch_Keyboard:SW_Cherry_MX_1.00u_PCB, symbol Switch:SW_Push
- removed SW58: LCtrl, Button_Switch_Keyboard:SW_Cherry_MX_1.00u_PCB, symbol Switch:SW_Push
- removed SW59: LWin, Button_Switch_Keyboard:SW_Cherry_MX_1.00u_PCB, symbol Switch:SW_Push
- removed SW6: 5, Button_Switch_Keyboard:SW_Cherry_MX_1.00u_PCB, symbol Switch:SW_Push
- removed SW60: LAlt, Button_Switch_Keyboard:SW_Cherry_MX_1.00u_PCB, symbol Switch:SW_Push
- removed SW61: Space625, Button_Switch_Keyboard:SW_Cherry_MX_1.00u_PCB, symbol Switch:SW_Push
- removed SW62: Space225, Button_Switch_Keyboard:SW_Cherry_MX_1.00u_PCB, symbol Switch:SW_Push
- removed SW63: Space125, Button_Switch_Keyboard:SW_Cherry_MX_1.00u_PCB, symbol Switch:SW_Push
- removed SW64: Space275, Button_Switch_Keyboard:SW_Cherry_MX_1.00u_PCB, symbol Switch:SW_Push
- removed SW65: RAlt, Button_Switch_Keyboard:SW_Cherry_MX_1.00u_PCB, symbol Switch:SW_Push
- removed SW66: RWin, Button_Switch_Keyboard:SW_Cherry_MX_1.00u_PCB, symbol Switch:SW_Push
- removed SW67: Menu, Button_Switch_Keyboard:SW_Cherry_MX_1.00u_PCB, symbol Switch:SW_Push
- removed SW68: RCtrl, Button_Switch_Keyboard:SW_Cherry_MX_1.00u_PCB, symbol Switch:SW_Push
- removed SW69: Left, Button_Switch_Keyboard:SW_Cherry_MX_1.00u_PCB, symbol Switch:SW_Push
- removed SW7: 6, Button_Switch_Keyboard:SW_Cherry_MX_1.00u_PCB, symbol Switch:SW_Push
- removed SW70: Down, Button_Switch_Keyboard:SW_Cherry_MX_1.00u_PCB, symbol Switch:SW_Push
- removed SW71: Right, Button_Switch_Keyboard:SW_Cherry_MX_1.00u_PCB, symbol Switch:SW_Push
- removed SW8: 7, Button_Switch_Keyboard:SW_Cherry_MX_1.00u_PCB, symbol Switch:SW_Push
- removed SW9: 8, Button_Switch_Keyboard:SW_Cherry_MX_1.00u_PCB, symbol Switch:SW_Push
- added C18, C19, C20, C21, C22, C23, C24, C25, C26, C27, C28, C29, C30, C31, C32, C33, C34, C35, C36, C37, C38, C39, C40, C41, C42, C43, C44, C45, C46, C47, C48, C49, C50, C51, C52, C53, C54, C55, C56, C57, C58, C59, C60, C61, C62, C63, C64, C65, C66, C67, C68, C69, C70, C71, C72, C73, C74, C75, C76, C77: 100n, Capacitor_SMD:C_0603_1608Metric, symbol Device:C
- added D62: RED, LED_SMD:LED_0603_1608Metric, symbol Device:LED
- added H1: MountingHole, lib.pretty:PKRHC, symbol Mechanical:MountingHole
- added H2, H4, H6: MountingHole, lib.pretty:PKRH, symbol Mechanical:MountingHole
- added H3, H5: MountingHole, lib.pretty:PKRHSL, symbol Mechanical:MountingHole
- added H7: MountingHole, lib.pretty:KB_BlueMicro, symbol Mechanical:MountingHole
- added J1: USB_C_Receptacle_USB2.0, Connector_USB:USB_C_Receptacle_HRO_TYPE-C-31-M-12, symbol Connector:USB_C_Receptacle_USB2.0
- added J2: Conn_01x03, Connector_PinHeader_2.54mm:PinHeader_1x03_P2.54mm_Vertical, symbol Connector_Generic:Conn_01x03
- added J3: Conn_01x04, Connector_PinHeader_2.54mm:PinHeader_1x04_P2.54mm_Vertical, symbol Connector_Generic:Conn_01x04
- added J4: Conn_01x06, Connector_PinHeader_2.54mm:PinHeader_1x06_P2.54mm_Vertical, symbol Connector_Generic:Conn_01x06
- added LS1: Speaker, Buzzer_Beeper:Buzzer_Mallory_AST1109MLTRQ, symbol Device:Speaker
- added R7, R8: 1k, Resistor_SMD:R_0603_1608Metric, symbol Device:R
- added RGB1, RGB2: SK6812MINI-E, Keyboard RGB:RGB_SK6812MINI-E, symbol Keyboard Common:SK6812MINI-E
- added SW1: SW_SPST, Button_Switch_SMD:SW_Push_SPST_NO_Alps_SKRK, symbol Switch:SW_SPST
- added SW2: SW_SPDT, Button_Switch_SMD:SW_SPDT_PCM12, symbol Switch:SW_SPDT
- added SW3, SW4: CherryMX, Keyboard Switches:SW_MX_HotSwap_reinforced, symbol CherryMX:CherryMX
- added U1, U10, U11, U12, U13, U16, U17, U18, U19, U2, U20, U21, U22, U23, U24, U25, U26, U27, U3, U30, U31, U32, U33, U34, U35, U36, U37, U38, U39, U4, U40, U43, U44, U45, U46, U47, U48, U49, U5, U50, U51, U52, U6, U7, U8, U9: CherryMX_LTST-A683CEGBW, CherryMX_PCB_KailhSocket_LTST-A683CEGBW-Rotated-HS:CherryMX_1.00u_PCB_KailhSocket_LTST-A683CEGBW-Rotated-HS, symbol CherryMX:CherryMX_LTST-A683CEGBW
- added U14: CherryMX_LTST-A683CEGBW, CherryMX_PCB_KailhSocket_StabWireTop_LTST-A683CEGBW-Rotated-HS:CherryMX_2.00u_PCB_KailhSocket_StabWireTop_LTST-A683CEGB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, symbol CherryMX:CherryMX_LTST-A683CEGBW
- added U15, U28: CherryMX_LTST-A683CEGBW, CherryMX_PCB_KailhSocket_LTST-A683CEGBW-Rotated-HS:CherryMX_1.50u_PCB_KailhSocket_LTST-A683CEGBW-Rotated-HS, symbol CherryMX:CherryMX_LTST-A683CEGBW
- added U29: CherryMX_LTST-A683CEGBW, CherryMX_PCB_KailhSocket_LTST-A683CEGBW-Rotated-HS:CherryMX_1.75u_PCB_KailhSocket_LTST-A683CEGBW-Rotated-HS, symbol CherryMX:CherryMX_LTST-A683CEGBW
- added U41, U42: CherryMX_LTST-A683CEGBW, CherryMX_PCB_KailhSocket_StabWireBottom_LTST-A683CEGBW-Rotated-HS:CherryMX_2.25u_PCB_KailhSocket_StabWireBottom_LTST-A6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, symbol CherryMX:CherryMX_LTST-A683CEGBW
- added U53: CherryMX_LTST-A683CEGBW, CherryMX_PCB_KailhSocket_StabWireBottom_LTST-A683CEGBW-Rotated-HS:CherryMX_2.75u_PCB_KailhSocket_StabWireBottom_LTST-A6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, symbol CherryMX:CherryMX_LTST-A683CEGBW
- added U54, U55, U56, U58, U59, U60, U61: CherryMX_LTST-A683CEGBW, CherryMX_PCB_KailhSocket_LTST-A683CEGBW-Rotated-HS:CherryMX_1.25u_PCB_KailhSocket_LTST-A683CEGBW-Rotated-HS, symbol CherryMX:CherryMX_LTST-A683CEGBW
- added U57: CherryMX_LTST-A683CEGBW, CherryMX_PCB_KailhSocket_StabWireBottom_LTST-A683CEGBW-Rotated-HS:CherryMX_6.25u_PCB_KailhSocket_StabWireBottom_LTST-A6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, symbol CherryMX:CherryMX_LTST-A683CEGBW
- added U62: RP2040, RP2040_minimal:RP2040-QFN-56, symbol MCU_RaspberryPi_RP2040:RP2040
- added U63: USBLC6-2SC6, Package_TO_SOT_SMD:SOT-23-6, symbol Power_Protection:USBLC6-2SC6
- added U64: W25Q128JVS, Package_SO:SOIC-8_5.23x5.23mm_P1.27mm, symbol Memory_Flash:W25Q128JVS
- added U65: AMS1117-3.3, Package_TO_SOT_SMD:SOT-223-3_TabPin2, symbol Regulator_Linear:AMS1117-3.3
- added Y1: 12MHz, Crystal:Crystal_SMD_3225-4Pin_3.2x2.5mm, symbol Device:Crystal_GND24_Small
- C1, C2: value 10uF -> 100n; footprint Capacitor_SMD:C_0805_2012Metric -> Capacitor_SMD:C_0603_1608Metric; LCSC (none) -> C14663
- C10: value 100nF -> 1u; footprint Capacitor_SMD:C_0402_1005Metric -> Capacitor_SMD:C_0603_1608Metric; LCSC (none) -> C15849
- C11: value 1uF -> 1u; footprint Capacitor_SMD:C_0402_1005Metric -> Capacitor_SMD:C_0603_1608Metric; LCSC (none) -> C15849
- C12: value 100nF -> 22p; footprint Capacitor_SMD:C_0402_1005Metric -> Capacitor_SMD:C_0603_1608Metric; LCSC (none) -> C1653
- C13: value 1uF -> 22p; footprint Capacitor_SMD:C_0402_1005Metric -> Capacitor_SMD:C_0603_1608Metric; LCSC (none) -> C1653
- C14: value 20pF -> 100n; footprint Capacitor_SMD:C_0402_1005Metric -> Capacitor_SMD:C_0603_1608Metric; LCSC (none) -> C14663
- C15: value 20pF -> 22u; footprint Capacitor_SMD:C_0402_1005Metric -> Capacitor_SMD:C_0603_1608Metric; LCSC (none) -> C59461
- C16: value 100nF -> 22u; footprint Capacitor_SMD:C_0402_1005Metric -> Capacitor_SMD:C_0603_1608Metric; LCSC (none) -> C59461
- C17, C3, C4, C5, C6, C7, C8, C9: value 100nF -> 100n; footprint Capacitor_SMD:C_0402_1005Metric -> Capacitor_SMD:C_0603_1608Metric; LCSC (none) -> C14663
- D1, D10, D11, D12, D13, D14, D15, D16, D17, D18, D19, D2, D20, D21, D22, D23, D24, D25, D26, D27, D28, D29, D3, D30, D31, D32, D33, D34, D35, D36, D37, D38, D39, D4, D40, D41, D42, D43, D44, D45, D46, D47, D48, D49, D5, D50, D51, D52, D53, D54, D55, D56, D57, D58, D59, D6, D60, D61, D63, D7, D8, D9: value 1N4148W -> D
- R1, R2: footprint Resistor_SMD:R_0402_1005Metric -> Resistor_SMD:R_0603_1608Metric; LCSC (none) -> C23186
- R3: value 1M -> 22; footprint Resistor_SMD:R_0402_1005Metric -> Resistor_SMD:R_0603_1608Metric; LCSC (none) -> C23345
- R4: value 10k -> 22; footprint Resistor_SMD:R_0402_1005Metric -> Resistor_SMD:R_0603_1608Metric; LCSC (none) -> C23345
- R5: value 10k -> 1k; footprint Resistor_SMD:R_0402_1005Metric -> Resistor_SMD:R_0603_1608Metric; LCSC (none) -> C21190
- R6: value 10k -> DNP; footprint Resistor_SMD:R_0402_1005Metric -> Resistor_SMD:R_0603_1608Metric
Connections:
- net CC1 is gone; now on net GND: R1.1
- net CC2 is gone; now on net GND: R2.1
- net VREG_OUT is gone; now on an unnamed net: C13.1
- net COL1: now also U1.2, U15.2, U29.2, U42.2, U54.2, U62.2 (GPIO0)
- net COL10: now also U10.2, U24.2, U38.2, U51.2, U58.2, U62.12 (GPIO9)
- net COL11: now also U11.2, U25.2, U39.2, U52.2, U59.2, U62.13 (GPIO10)
- net COL12: now also U12.2, U26.2, U40.2, U60.2, U62.14 (GPIO11)
- net COL13: now also U13.2, U27.2, U62.15 (GPIO12)
- net COL14: now also SW3.2, U14.2, U28.2, U41.2, U53.2, U61.2, U62.16 (GPIO13)
- net COL2: now also U16.2, U2.2, U30.2, U43.2, U55.2, U62.3 (GPIO1)
- net COL3: now also U17.2, U3.2, U31.2, U44.2, U56.2, U62.4 (GPIO2)
- net COL4: now also U18.2, U32.2, U4.2, U45.2, U62.5 (GPIO3)
- net COL5: now also U19.2, U33.2, U46.2, U5.2, U62.6 (GPIO4)
- net COL6: now also U20.2, U34.2, U47.2, U57.2, U6.2, U62.7 (GPIO5)
- net COL7: now also U21.2, U35.2, U48.2, U62.8 (GPIO6), U7.2
- net COL8: now also U22.2, U36.2, U49.2, U62.9 (GPIO7), U8.2
- net COL9: now also U23.2, U37.2, U50.2, U62.11 (GPIO8), U9.2
- net GND: now also C18.2, C19.2, C20.2, C21.2, C22.2, C23.2, C24.2, C25.2, C26.2, C27.2, C28.2, C29.2, C30.2, C31.2, C32.2, C33.2, C34.2, C35.2, C36.2, C37.2, C38.2, C39.2, C40.2, C41.2, C42.2, C43.2, C44.2, C45.2, C46.2, C47.2, C48.2, C49.2, C50.2, C51.2, C52.2, C53.2, C54.2, C55.2, C56.2, C57.2, C58.2, C59.2, C60.2, C61.2, C62.2, C63.2, C64.2, C65.2, C66.2, C67.2, C68.2, C69.2, C70.2, C71.2, C72.2, C73.2, C74.2, C75.2, C76.2, C77.2, D62.1 (K), J1.A1 (GND), J1.A12 (GND), J1.B1 (GND), J1.B12 (GND), J2.2 (Pin_2), J3.4 (Pin_4), J4.6 (Pin_6), LS1.2, RGB1.3 (GND), RGB2.3 (GND), SW1.1 (A), SW2.2 (B), U1.3 (VSS), U10.3 (VSS), U11.3 (VSS), U12.3 (VSS), U13.3 (VSS), U14.3 (VSS), U15.3 (VSS), U16.3 (VSS), U17.3 (VSS), U18.3 (VSS), U19.3 (VSS), U2.3 (VSS), U20.3 (VSS), U21.3 (VSS), U22.3 (VSS), U23.3 (VSS), U24.3 (VSS), U25.3 (VSS), U26.3 (VSS), U27.3 (VSS), U28.3 (VSS), U29.3 (VSS), U3.3 (VSS), U30.3 (VSS), U31.3 (VSS), U32.3 (VSS), U33.3 (VSS), U34.3 (VSS), U35.3 (VSS), U36.3 (VSS), U37.3 (VSS), U38.3 (VSS), U39.3 (VSS), U4.3 (VSS), U40.3 (VSS), U41.3 (VSS), U42.3 (VSS), U43.3 (VSS), U44.3 (VSS), U45.3 (VSS), U46.3 (VSS), U47.3 (VSS), U48.3 (VSS), U49.3 (VSS), U5.3 (VSS), U50.3 (VSS), U51.3 (VSS), U52.3 (VSS), U53.3 (VSS), U54.3 (VSS), U55.3 (VSS), U56.3 (VSS), U57.3 (VSS), U58.3 (VSS), U59.3 (VSS), U6.3 (VSS), U60.3 (VSS), U61.3 (VSS), U62.19 (TESTEN), U62.57 (GND), U64.4 (GND), U65.1 (GND), U7.3 (VSS), U8.3 (VSS), U9.3 (VSS), Y1.2 (G), Y1.4 (G); no longer R1.2, R2.2
- net ROW1: now also D1.1 (K), D10.1 (K), D11.1 (K), D12.1 (K), D13.1 (K), D14.1 (K), D2.1 (K), D3.1 (K), D4.1 (K), D5.1 (K), D6.1 (K), D7.1 (K), D8.1 (K), D9.1 (K), U62.17 (GPIO14); no longer D16.2 (A), D17.2 (A), D18.2 (A), D19.2 (A), D20.2 (A), D21.2 (A), D22.2 (A), D23.2 (A), D24.2 (A), D25.2 (A), D26.2 (A), D27.2 (A), D28.2 (A), D29.2 (A), D30.2 (A)
- net ROW2: now also D15.1 (K), D16.1 (K), D17.1 (K), D18.1 (K), D19.1 (K), D20.1 (K), D21.1 (K), D22.1 (K), D23.1 (K), D24.1 (K), D25.1 (K), D26.1 (K), D27.1 (K), D28.1 (K), U62.18 (GPIO15); no longer D31.2 (A), D32.2 (A), D33.2 (A), D34.2 (A), D35.2 (A), D36.2 (A), D37.2 (A), D38.2 (A), D39.2 (A), D40.2 (A), D41.2 (A), D42.2 (A), D43.2 (A)
- net ROW3: now also D29.1 (K), D30.1 (K), D31.1 (K), D32.1 (K), D33.1 (K), D34.1 (K), D35.1 (K), D36.1 (K), D37.1 (K), D38.1 (K), D39.1 (K), D40.1 (K), D41.1 (K), U62.27 (GPIO16); no longer D44.2 (A), D45.2 (A), D46.2 (A), D47.2 (A), D48.2 (A), D49.2 (A), D50.2 (A), D51.2 (A), D52.2 (A), D53.2 (A), D54.2 (A), D55.2 (A), D56.2 (A), D57.2 (A)
- net ROW4: now also D42.1 (K), D43.1 (K), D44.1 (K), D45.1 (K), D46.1 (K), D47.1 (K), D48.1 (K), D49.1 (K), D50.1 (K), D51.1 (K), D52.1 (K), D53.1 (K), U62.28 (GPIO17); no longer D58.2 (A), D59.2 (A), D60.2 (A), D61.2 (A), D63.2 (A)
- net VBUS: now also C15.1, J1.A4 (VBUS), J1.A9 (VBUS), J1.B4 (VBUS), J1.B9 (VBUS), U65.3 (VI); no longer C1.1
- net XIN: now also C12.1, U62.20 (XIN), Y1.1; no longer C14.1, R3.1
- net XOUT: now also R5.1, U62.21 (XOUT); no longer C15.1, R3.2
- net ROW5: now reaches D56.1 (K)
- net ROW5: now also D54.1 (K), D55.1 (K), D57.1 (K), D58.1 (K), D59.1 (K), D60.1 (K), D61.1 (K), U62.29 (GPIO18)
- net +3V3: now reaches R6.2
- net +3V3: now also C11.1, C14.1, C16.1, C17.1, C3.1, C4.1, C5.1, C6.1, C7.1, C8.1, C9.1, C18.1, C19.1, C20.1, C21.1, C22.1, C23.1, C24.1, C25.1, C26.1, C27.1, C28.1, C29.1, C30.1, C31.1, C32.1, C33.1, C34.1, C35.1, C36.1, C37.1, C38.1, C39.1, C40.1, C41.1, C42.1, C43.1, C44.1, C45.1, C46.1, C47.1, C48.1, C49.1, C50.1, C51.1, C52.1, C53.1, C54.1, C55.1, C56.1, C57.1, C58.1, C59.1, C60.1, C61.1, C62.1, C63.1, C64.1, C65.1, C66.1, C67.1, C68.1, C69.1, C70.1, C71.1, C72.1, C73.1, C74.1, C75.1, C76.1, C77.1, J3.3 (Pin_3), J4.5 (Pin_5), RGB1.1 (VDD), RGB2.1 (VDD), U1.6 (VDD), U10.6 (VDD), U11.6 (VDD), U12.6 (VDD), U13.6 (VDD), U14.6 (VDD), U15.6 (VDD), U16.6 (VDD), U17.6 (VDD), U18.6 (VDD), U19.6 (VDD), U2.6 (VDD), U20.6 (VDD), U21.6 (VDD), U22.6 (VDD), U23.6 (VDD), U24.6 (VDD), U25.6 (VDD), U26.6 (VDD), U27.6 (VDD), U28.6 (VDD), U29.6 (VDD), U3.6 (VDD), U30.6 (VDD), U31.6 (VDD), U32.6 (VDD), U33.6 (VDD), U34.6 (VDD), U35.6 (VDD), U36.6 (VDD), U37.6 (VDD), U38.6 (VDD), U39.6 (VDD), U4.6 (VDD), U40.6 (VDD), U41.6 (VDD), U42.6 (VDD), U43.6 (VDD), U44.6 (VDD), U45.6 (VDD), U46.6 (VDD), U47.6 (VDD), U48.6 (VDD), U49.6 (VDD), U5.6 (VDD), U50.6 (VDD), U51.6 (VDD), U52.6 (VDD), U53.6 (VDD), U54.6 (VDD), U55.6 (VDD), U56.6 (VDD), U57.6 (VDD), U58.6 (VDD), U59.6 (VDD), U6.6 (VDD), U60.6 (VDD), U61.6 (VDD), U62.1 (IOVDD), U62.10 (IOVDD), U62.22 (IOVDD), U62.33 (IOVDD), U62.42 (IOVDD), U62.43 (ADC_AVDD), U62.44 (VREG_IN), U62.48 (USB_VDD), U62.49 (IOVDD), U64.8 (VCC), U65.2 (VO), U7.6 (VDD), U8.6 (VDD), U9.6 (VDD)
- net at R5.2: now also Y1.3
- net at D63.1 (K): now also U40.5 (DOUT)
- removed net 3V3: C10.1, C11.1, C12.1, C16.1, C2.1, C3.1, C4.1, C5.1, C6.1, C7.1, C8.1, C9.1, R4.1, R5.1, R6.1
- removed net ROW0: D1.2 (A), D10.2 (A), D11.2 (A), D12.2 (A), D13.2 (A), D14.2 (A), D15.2 (A), D2.2 (A), D3.2 (A), D4.2 (A), D5.2 (A), D6.2 (A), D7.2 (A), D8.2 (A), D9.2 (A)
- net RUN: no longer names the net of R4.2
- net RUN: now also U62.46 (USB_DM); no longer C17.1
- new net: D1.2 (A), U1.1
- new net: U1.5 (DOUT), U2.4 (DIN)
- new net: D2.2 (A), U2.1
- new net: U2.5 (DOUT), U3.4 (DIN)
- new net: D3.2 (A), U3.1
- new net: U3.5 (DOUT), U4.4 (DIN)
- new net: D4.2 (A), U4.1
- new net: U4.5 (DOUT), U5.4 (DIN)
- new net: D5.2 (A), U5.1
- new net: U5.5 (DOUT), U6.4 (DIN)
- new net: D6.2 (A), U6.1
- new net: U6.5 (DOUT), U7.4 (DIN)
- new net: D7.2 (A), U7.1
- new net: U7.5 (DOUT), U8.4 (DIN)
- new net: D8.2 (A), U8.1
- new net: U8.5 (DOUT), U9.4 (DIN)
- new net: D9.2 (A), U9.1
- new net: U10.4 (DIN), U9.5 (DOUT)
- new net: D10.2 (A), U10.1
- new net: U10.5 (DOUT), U11.4 (DIN)
- new net: D11.2 (A), U11.1
- new net: U11.5 (DOUT), U12.4 (DIN)
- new net: D12.2 (A), U12.1
- new net: U12.5 (DOUT), U13.4 (DIN)
- new net: D13.2 (A), U13.1
- new net: U13.5 (DOUT), U14.4 (DIN)
- new net: D14.2 (A), SW3.1, U14.1
- new net: D15.2 (A), U15.1
- new net: U15.5 (DOUT), U16.4 (DIN)
- new net: D16.2 (A), U16.1
- new net: U16.5 (DOUT), U17.4 (DIN)
- new net: D17.2 (A), U17.1
- new net: U17.5 (DOUT), U18.4 (DIN)
- new net: D18.2 (A), U18.1
- new net: U18.5 (DOUT), U19.4 (DIN)
- new net: D19.2 (A), U19.1
- new net: U19.5 (DOUT), U20.4 (DIN)
- new net: D20.2 (A), U20.1
- new net: U20.5 (DOUT), U21.4 (DIN)
- new net: D21.2 (A), U21.1
- new net: U21.5 (DOUT), U22.4 (DIN)
- new net: D22.2 (A), U22.1
- new net: U22.5 (DOUT), U23.4 (DIN)
- new net: D23.2 (A), U23.1
- new net: U23.5 (DOUT), U24.4 (DIN)
- new net: D24.2 (A), U24.1
- new net: U24.5 (DOUT), U25.4 (DIN)
- new net: D25.2 (A), U25.1
- new net: U25.5 (DOUT), U26.4 (DIN)
- new net: D26.2 (A), U26.1
- new net: U26.5 (DOUT), U27.4 (DIN)
- new net: D27.2 (A), U27.1
- new net: U27.5 (DOUT), U28.4 (DIN)
- new net: D28.2 (A), U28.1
- new net: D29.2 (A), U29.1
- new net: U29.5 (DOUT), U30.4 (DIN)
- new net: D30.2 (A), U30.1
- new net: U30.5 (DOUT), U31.4 (DIN)
- new net: D31.2 (A), U31.1
- new net: U31.5 (DOUT), U32.4 (DIN)
- new net: D32.2 (A), U32.1
- new net: U32.5 (DOUT), U33.4 (DIN)
- new net: D33.2 (A), U33.1
- new net: U33.5 (DOUT), U34.4 (DIN)
- new net: D34.2 (A), U34.1
- new net: U34.5 (DOUT), U35.4 (DIN)
- new net: D35.2 (A), U35.1
- new net: U35.5 (DOUT), U36.4 (DIN)
- new net: D36.2 (A), U36.1
- new net: U36.5 (DOUT), U37.4 (DIN)
- new net: D37.2 (A), U37.1
- new net: U37.5 (DOUT), U38.4 (DIN)
- new net: D38.2 (A), U38.1
- new net: U38.5 (DOUT), U39.4 (DIN)
- new net: D39.2 (A), U39.1
- new net: U39.5 (DOUT), U40.4 (DIN)
- new net: D40.2 (A), U40.1
- new net: D41.2 (A), U41.1
- new net: SW4.2, U41.4 (DIN)
- new net: D42.2 (A), U42.1
- new net: U42.5 (DOUT), U43.4 (DIN)
- new net: D43.2 (A), U43.1
- new net: U43.5 (DOUT), U44.4 (DIN)
- new net: D44.2 (A), U44.1
- new net: U44.5 (DOUT), U45.4 (DIN)
- new net: D45.2 (A), U45.1
- new net: U45.5 (DOUT), U46.4 (DIN)
- new net: D46.2 (A), U46.1
- new net: U46.5 (DOUT), U47.4 (DIN)
- new net: D47.2 (A), U47.1
- new net: U47.5 (DOUT), U48.4 (DIN)
- new net: D48.2 (A), U48.1
- new net: U48.5 (DOUT), U49.4 (DIN)
- new net: D49.2 (A), U49.1
- new net: U49.5 (DOUT), U50.4 (DIN)
- new net: D50.2 (A), U50.1
- new net: U50.5 (DOUT), U51.4 (DIN)
- new net: D51.2 (A), U51.1
- new net: U51.5 (DOUT), U52.4 (DIN)
- new net: D52.2 (A), U52.1
- new net: U52.5 (DOUT), U53.4 (DIN)
- new net: D53.2 (A), U53.1
- new net: D54.2 (A), U54.1
- new net: U54.5 (DOUT), U55.4 (DIN)
- new net: D55.2 (A), U55.1
- new net: U55.5 (DOUT), U56.4 (DIN)
- new net: D56.2 (A), U56.1
- new net: U56.5 (DOUT), U57.4 (DIN)
- new net: D57.2 (A), U57.1
- new net: U57.5 (DOUT), U58.4 (DIN)
- new net: D58.2 (A), U58.1
- new net: U58.5 (DOUT), U59.4 (DIN)
- new net: D59.2 (A), U59.1
- new net: U59.5 (DOUT), U60.4 (DIN)
- new net: D60.2 (A), U60.1
- new net: U60.5 (DOUT), U61.4 (DIN)
- new net: D61.2 (A), U61.1
- new net: J1.A5 (CC1), R1.2
- new net: J1.B5 (CC2), R2.2
- new net: R3.2, U62.47 (USB_DP)
- new net: R7.2, SW2.3 (C)
- new net: D62.2 (A), R8.1
- new net: RGB1.2 (DOUT), RGB2.4 (DIN)
- new net: D63.2 (A), SW4.1
- new net +1V1: C1.1, C10.1, C2.1, U62.23 (DVDD), U62.45 (VREG_VOUT), U62.50 (DVDD)
- new net Data+: R3.1
- new net Data-: R4.1
- new net I2C1_SCL: J3.1 (Pin_1), U62.35 (GPIO23)
- new net I2C1_SDA: J3.2 (Pin_2), U62.34 (GPIO22)
- new net LED: R8.2, U62.36 (GPIO24)
- new net QSPICLK: U62.52 (QSPI_SCLK)
- new net QSPISD0: U62.53 (QSPI_SD0)
- new net QSPISD2: U62.54 (QSPI_SD2)
- new net QSPISD3: U62.51 (QSPI_SD3)
- new net QSPISS: R6.1, R7.1, U62.56 (QSPI_SS)
- new net RESET: SW1.2 (B), U62.26 (RUN)
- new net RGBData1: U1.4 (DIN), U62.41 (GPIO29_ADC3)
- new net RGBData2: RGB2.2 (DOUT), U15.4 (DIN)
- new net RGBData3: U28.5 (DOUT), U29.4 (DIN)
- new net RGBData4: U41.5 (DOUT), U42.4 (DIN)
- new net RGBData5: U53.5 (DOUT), U54.4 (DIN)
- new net RGBEXT: RGB1.4 (DIN), U14.5 (DOUT)
- new net SPEAKER: LS1.1, U62.32 (GPIO21)
- new net SPI1_CSn: J4.1 (Pin_1), U62.37 (GPIO25)
- new net SPI1_RX: J4.4 (Pin_4), U62.40 (GPIO28_ADC2)
- new net SPI1_SCK: J4.2 (Pin_2), U62.38 (GPIO26_ADC0)
- new net SPI1_TX: J4.3 (Pin_3), U62.39 (GPIO27_ADC1)
- new net SQPISD1: U62.55 (QSPI_SD1)
- new net SWCLK: J2.3 (Pin_3), U62.24 (SWCLK)
- new net SWD: J2.1 (Pin_1), U62.25 (SWD)
- new net USB+: J1.A6 (D+), J1.B6 (D+)
- new net USB-: J1.A7 (D-), J1.B7 (D-)
- no-connect marks 0 -> 7
Other:
- note removed: "12MHz CRYSTAL (Y1)"
- note removed: "2-layer: F.Cu + B.Cu | GND planes both sides"
- note removed: "5 rows x 15 columns | Diodes: cathode to ROW"
- note removed: "<- GP0 (row output)"
- note removed: "<- GP1 (row output)"
- note removed: "<- GP10 (col input, pullup)"
- note removed: "<- GP11 (col input, pullup)"
- note removed: "<- GP12 (col input, pullup)"
- note removed: "<- GP13 (col input, pullup)"
- note removed: "<- GP14 (col input, pullup)"
- note removed: "<- GP15 (col input, pullup)"
- note removed: "<- GP16 (col input, pullup)"
- note removed: "<- GP17 (col input, pullup)"
- note removed: "<- GP18 (col input, pullup)"
- note removed: "<- GP19 (col input, pullup)"
- note removed: "<- GP2 (row output)"
- note removed: "<- GP3 (row output)"
- note removed: "<- GP4 (row output)"
- note removed: "<- GP5 (col input, pullup)"
- note removed: "<- GP6 (col input, pullup)"
- note removed: "<- GP7 (col input, pullup)"
- note removed: "<- GP8 (col input, pullup)"
- note removed: "<- GP9 (col input, pullup)"
- note removed: "ADC_AVDD"
- note removed: "ADC_AVDD: -> 100nF (C12)"
- note removed: "BOM SUMMARY"
- note removed: "Board: 285.0mm x 94.5mm | USB-C top-left"
- note removed: "Bypass"
- note removed: "C1,C2: 10uF | C3-C12,C16,C17: 100nF"
- note removed: "C11,C13: 1uF | C14,C15: 20pF"
- note removed: "CS->QSPI_SS_N CLK->QSPI_SCLK"
- note removed: "Column Inputs:"
- note removed: "D1-D71: 1N4148W SOD-123"
- note removed: "DVDD (x6): -> 100nF each (C4-C9)"
- note removed: "DVDD1"
- note removed: "DVDD2"
- note removed: "DVDD3"
- note removed: "DVDD4"
- note removed: "DVDD5"
- note removed: "DVDD6"
- note removed: "F1: 500mA PTC fuse on VBUS"
- note removed: "Firmware: QMK (RP2040 native support)"
- note removed: "GPIO Pin Assignments:"
- note removed: "GPIO: 20/30 used, 10 free"
- note removed: "Hold BOOT + RESET = UF2 bootloader"
- note removed: "IO0->QSPI_SD0 IO1->QSPI_SD1"
- note removed: "IO2 pullup"
- note removed: "IO2->QSPI_SD2 (R5 10k pullup)"
- note removed: "IO3 pullup"
- note removed: "IO3->QSPI_SD3 (R6 10k pullup)"
- note removed: "J1: USB-C mid-mount"
- note removed: "Matrix: 5R x 15C = 71 switches"
- note removed: "Mid-mount | Top-left of PCB (285x94.5mm)"
- note removed: "NO VIAS between crystal and MCU!"
- note removed: "Other RP2040 Connections:"
- note removed: "PCB DESIGN NOTES"
- note removed: "POWER (U2: AP2112K-3.3)"
- note removed: "QFN-56 | GPIO directly mapped to matrix"
- note removed: "QSPI FLASH (U4: W25Q128JVS)"
- note removed: "QSPI_SS, SCLK, SD0-3: -> Flash U4"
- note removed: "R1,R2: 5.1k | R3: 1M | R4-R6: 10k"
- note removed: "RESET & BOOT"
- note removed: "RP2040 Decoupling:"
- note removed: "RP2040 MICROCONTROLLER (U1)"
- note removed: "RUN: -> Reset (R4 pullup + SW_RST)"
- note removed: "Route: crystal first, then VCC, USB, power, matrix"
- note removed: "SW1-SW71: MX + Kailh hot-swap socket"
- note removed: "SWITCH MATRIX"
- note removed: "SW_BOOT: QSPI_SS -> switch -> GND"
- note removed: "SW_RST: RUN -> switch -> GND"
- note removed: "Switches on front | Everything else on back"
- note removed: "U1: RP2040 QFN-56"
- note removed: "U2: AP2112K-3.3 SOT-23-5"
- note removed: "U3: USBLC6-2SC6 (ESD on D+/D-)"
- note removed: "U3: USBLC6-2SC6 SOT-23-6"
- note removed: "U4: W25Q128JVS SOIC-8"
- note removed: "USB-C CONNECTOR (J1)"
- note removed: "USB_DP / USB_DM: Internal USB PHY"
- note removed: "USB_VDD"
- note removed: "USB_VDD: -> 100nF+1uF (C10,C11)"
- note removed: "USB_VDD_bulk"
- note removed: "VCC->3V3 GND->GND"
- note removed: "VIN filter"
- note removed: "VOUT filter"
- note removed: "VREG_VIN -> 3V3: VREG_VOUT -> 1uF (C13)"
- note removed: "VREG_VOUT"
- note removed: "XIN/XOUT (dedicated): -> Crystal Y1"
- note removed: "Y1: 12MHz crystal 3215"
- company: (none) -> Pierre Constantineau (JPConstantineau)
- title: Custom 65%% Keyboard - RP2040 -> PyKey60 RP2040
