File: 60rtho.kicad_sch (KiCad schematic)
At the start: 232 parts, among them J1 USB_C_Receptacle_USB2.0, J2 Conn_01x03, J3 Conn_01x04, J4 Conn_01x06, SW1 SW_SPST, SW2 SW_SPDT, SW3 CherryMX, SW4 CherryMX, U1 CherryMX_LTST-A683CEGBW, U10 CherryMX_LTST-A683CEGBW, U11 CherryMX_LTST-A683CEGBW, U12 CherryMX_LTST-A683CEGBW, U13 CherryMX_LTST-A683CEGBW, U14 CherryMX_LTST-A683CEGBW, U15 CherryMX_LTST-A683CEGBW, U16 CherryMX_LTST-A683CEGBW, U17 CherryMX_LTST-A683CEGBW, U18 CherryMX_LTST-A683CEGBW, U19 CherryMX_LTST-A683CEGBW, U2 CherryMX_LTST-A683CEGBW, U20 CherryMX_LTST-A683CEGBW, U21 CherryMX_LTST-A683CEGBW, U22 CherryMX_LTST-A683CEGBW, U23 CherryMX_LTST-A683CEGBW, U24 CherryMX_LTST-A683CEGBW, U25 CherryMX_LTST-A683CEGBW, U26 CherryMX_LTST-A683CEGBW, U27 CherryMX_LTST-A683CEGBW, U28 CherryMX_LTST-A683CEGBW, U29 CherryMX_LTST-A683CEGBW, U3 CherryMX_LTST-A683CEGBW, U30 CherryMX_LTST-A683CEGBW, U31 CherryMX_LTST-A683CEGBW, U32 CherryMX_LTST-A683CEGBW, U33 CherryMX_LTST-A683CEGBW, U34 CherryMX_LTST-A683CEGBW, U35 CherryMX_LTST-A683CEGBW, U36 CherryMX_LTST-A683CEGBW, U37 CherryMX_LTST-A683CEGBW, U38 CherryMX_LTST-A683CEGBW, U39 CherryMX_LTST-A683CEGBW, U4 CherryMX_LTST-A683CEGBW, U40 CherryMX_LTST-A683CEGBW, U41 CherryMX_LTST-A683CEGBW, U42 CherryMX_LTST-A683CEGBW, U43 CherryMX_LTST-A683CEGBW, U44 CherryMX_LTST-A683CEGBW, U45 CherryMX_LTST-A683CEGBW, U46 CherryMX_LTST-A683CEGBW, U47 CherryMX_LTST-A683CEGBW, U48 CherryMX_LTST-A683CEGBW, U49 CherryMX_LTST-A683CEGBW, U5 CherryMX_LTST-A683CEGBW, U50 CherryMX_LTST-A683CEGBW, U51 CherryMX_LTST-A683CEGBW, U52 CherryMX_LTST-A683CEGBW, U53 CherryMX_LTST-A683CEGBW, U54 CherryMX_LTST-A683CEGBW, U55 CherryMX_LTST-A683CEGBW, U56 CherryMX_LTST-A683CEGBW, U57 CherryMX_LTST-A683CEGBW, U58 CherryMX_LTST-A683CEGBW, U59 CherryMX_LTST-A683CEGBW, U6 CherryMX_LTST-A683CEGBW, U60 CherryMX_LTST-A683CEGBW, U61 CherryMX_LTST-A683CEGBW, U62 RP2040, U63 USBLC6-2SC6, U64 W25Q128JVS, U65 AMS1117-3.3, U7 CherryMX_LTST-A683CEGBW, U8 CherryMX_LTST-A683CEGBW, U9 CherryMX_LTST-A683CEGBW, Y1 12MHz

Commit message: adjusted schematics and pcb
adjusted schematics and pcb
71 switches centered within the board ✓
Equal left/right margins ✓
All diodes positioned ✓
MCU and support circuitry intact ✓

The remaining work is routing the traces and verifying overlaps
Parts:
- added D64, D65, D66, D67, D68, D69, D70, D71, D72, D73: D, Diode_SMD:D_SOD-123, symbol Device:D
- added U66, U68, U73, U74, U75: CherryMX_LTST-A683CEGBW, CherryMX_PCB_KailhSocket_LTST-A683CEGBW-Rotated-HS:CherryMX_1.00u_PCB_KailhSocket_LTST-A683CEGBW-Rotated-HS, symbol CherryMX:CherryMX_LTST-A683CEGBW
- added U67: CherryMX_LTST-A683CEGBW, CherryMX_PCB_KailhSocket_LTST-A683CEGBW-Rotated-HS:CherryMX_1.50u_PCB_KailhSocket_LTST-A683CEGBW-Rotated-HS, symbol CherryMX:CherryMX_LTST-A683CEGBW
- added U69, U70: CherryMX_LTST-A683CEGBW, CherryMX_PCB_KailhSocket_StabWireBottom_LTST-A683CEGBW-Rotated-HS:CherryMX_2.25u_PCB_KailhSocket_StabWireBottom_LTST-A6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, symbol CherryMX:CherryMX_LTST-A683CEGBW
- added U71: CherryMX_LTST-A683CEGBW, CherryMX_PCB_KailhSocket_LTST-A683CEGBW-Rotated-HS:CherryMX_1.25u_PCB_KailhSocket_LTST-A683CEGBW-Rotated-HS, symbol CherryMX:CherryMX_LTST-A683CEGBW
- added U72: CherryMX_LTST-A683CEGBW, CherryMX_PCB_KailhSocket_StabWireBottom_LTST-A683CEGBW-Rotated-HS:CherryMX_2.75u_PCB_KailhSocket_StabWireBottom_LTST-A6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, symbol CherryMX:CherryMX_LTST-A683CEGBW
Connections:
- net COL13: now also U67.6 (VDD), U68.6 (VDD), U75.6 (VDD)
- net COL14: now also U66.6 (VDD), U69.6 (VDD)
- net COL4: now also U70.6 (VDD)
- net COL5: now also U71.6 (VDD)
- net COL7: now also U72.6 (VDD)
- net COL8: now also U73.6 (VDD)
- net COL9: now also U74.6 (VDD)
- net ROW1: now also D64.1 (K)
- net ROW2: now also D65.1 (K)
- net ROW4: now also D66.1 (K), D67.1 (K)
- net ROW5: now also D68.1 (K), D69.1 (K), D70.1 (K), D71.1 (K), D72.1 (K), D73.1 (K)
- new net: D71.2 (A), U73.4 (DIN)
- new net: D69.2 (A), U71.4 (DIN)
- new net: D72.2 (A), U74.4 (DIN)
- new net: D67.2 (A), U69.4 (DIN)
- new net: D73.2 (A), U75.4 (DIN)
- new net: D70.2 (A), U72.4 (DIN)
- new net: D65.2 (A), U67.4 (DIN)
- new net: D68.2 (A), U70.4 (DIN)
- new net: D64.2 (A), U66.4 (DIN)
- new net: D66.2 (A), U68.4 (DIN)

Commit message: Cleaned up
Removed excessive 100nF and accesories that make no sense.
Split RGB and Switches to different footprints.
Parts:
- removed C47, C48, C49, C50, C51, C52, C53, C54, C55, C56, C57, C58, C59, C60, C61, C62, C63, C64, C65, C66, C67, C68, C69, C70, C71, C72, C73, C74, C75, C76, C77: 100n, Capacitor_SMD:C_0603_1608Metric, symbol Device:C
- removed J3: Conn_01x04, Connector_PinHeader_2.54mm:PinHeader_1x04_P2.54mm_Vertical, symbol Connector_Generic:Conn_01x04
- removed J4: Conn_01x06, Connector_PinHeader_2.54mm:PinHeader_1x06_P2.54mm_Vertical, symbol Connector_Generic:Conn_01x06
- removed LS1: Speaker, Buzzer_Beeper:Buzzer_Mallory_AST1109MLTRQ, symbol Device:Speaker
Connections:
- net Data+: now also U63.6 (I/O1)
- net Data-: now also U63.1 (I/O1)
- net GND: now also U63.2 (GND)
- net LED: no longer U62.36 (GPIO24)
- net RGBData1: no longer U62.41 (GPIO29_ADC3)
- net USB+: now also U63.4 (I/O2)
- net USB-: now also U63.3 (I/O2)
- net VBUS: now also U63.5 (VBUS)
- net I2C1_SCL: no longer names the net of U62.35 (GPIO23)
- net I2C1_SDA: no longer names the net of U62.34 (GPIO22)
- net SPEAKER: no longer names the net of U62.32 (GPIO21)
- net SPI1_CSn: no longer names the net of U62.37 (GPIO25)
- net SPI1_RX: no longer names the net of U62.40 (GPIO28_ADC2)
- net SPI1_SCK: no longer names the net of U62.38 (GPIO26_ADC0)
- net SPI1_TX: no longer names the net of U62.39 (GPIO27_ADC1)
- no-connect marks 7 -> 16
Other:
- moved on the sheet: C1, C10, C11, C12, C13, C14, C15, C16, C17, C18, C19, C2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
