File: 60rtho.kicad_sch (KiCad schematic)
At the start: 289 parts, among them J1 USB_C_Receptacle_USB2.0, J2 Conn_01x03, SW1 SW_SPST, SW2 SW_SPDT, SW3 CherryMX, SW4 CherryMX, U1 CherryMX_LTST-A683CEGBW, U10 CherryMX_LTST-A683CEGBW, U100 RGB_(edited), U101 RGB_(edited), U102 RGB_(edited), U103 RGB_(edited), U104 RGB_(edited), U105 RGB_(edited), U106 RGB_(edited), U107 RGB_(edited), U108 RGB_(edited), U109 RGB_(edited), U11 CherryMX_LTST-A683CEGBW, U110 RGB_(edited), U111 RGB_(edited), U112 RGB_(edited), U113 RGB_(edited), U114 RGB_(edited), U115 RGB_(edited), U116 RGB_(edited), U117 RGB_(edited), U118 RGB_(edited), U119 RGB_(edited), U12 CherryMX_LTST-A683CEGBW, U120 RGB_(edited), U121 RGB_(edited), U122 RGB_(edited), U123 RGB_(edited), U124 RGB_(edited), U125 RGB_(edited), U126 RGB_(edited), U127 RGB_(edited), U128 RGB_(edited), U129 RGB_(edited), U13 CherryMX_LTST-A683CEGBW, U130 RGB_(edited), U131 RGB_(edited), U132 RGB_(edited), U133 RGB_(edited), U134 RGB_(edited), U135 RGB_(edited), U136 RGB_(edited), U137 RGB_(edited), U138 RGB_(edited), U139 RGB_(edited), U14 CherryMX_LTST-A683CEGBW, U140 RGB_(edited), U141 RGB_(edited), U142 RGB_(edited), U143 RGB_(edited), U144 RGB_(edited), U145 RGB_(edited), U146 RGB_(edited), U15 CherryMX_LTST-A683CEGBW, U16 CherryMX_LTST-A683CEGBW, U17 CherryMX_LTST-A683CEGBW, U18 CherryMX_LTST-A683CEGBW, U19 CherryMX_LTST-A683CEGBW, U2 CherryMX_LTST-A683CEGBW, U20 CherryMX_LTST-A683CEGBW, U21 CherryMX_LTST-A683CEGBW, U22 CherryMX_LTST-A683CEGBW, U23 CherryMX_LTST-A683CEGBW, U24 CherryMX_LTST-A683CEGBW, U25 CherryMX_LTST-A683CEGBW, U26 CherryMX_LTST-A683CEGBW, U27 CherryMX_LTST-A683CEGBW, U28 CherryMX_LTST-A683CEGBW, U29 CherryMX_LTST-A683CEGBW, U3 CherryMX_LTST-A683CEGBW, U30 CherryMX_LTST-A683CEGBW, U31 CherryMX_LTST-A683CEGBW, U32 CherryMX_LTST-A683CEGBW, U33 CherryMX_LTST-A683CEGBW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

Commit message: Place LEDs U76-U146 above their switches
Each LED placed 5.08mm above its switch, rotated 90° to match RGB1/RGB2.
Removed KiCad lock files and added .gitignore for *.lck and .history.
Other:
- company: Pierre Constantineau (JPConstantineau) -> Pedro Quaresma (TheReflex)
- title: PyKey60 RP2040 -> 60rtho RP2040
Changed lines of the file:
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@@
 	(paper "User" 524.9926 350.012)
 	(title_block
-		(title "PyKey60 RP2040")
-		(date "2021-09-16")
+		(title "60rtho RP2040")
+		(date "2026-10-19")
 		(rev "1.0")
-		(company "Pierre Constantineau (JPConstantineau)")
+		(company "Pedro Quaresma (TheReflex)")
 		(comment 1 "License: CERN-OHL-W (CERN OHL v2)")
-		(comment 2 "Project: https://github.com/jpconstantineau/PyKey60")
+		(comment 2 "Project: https://github.com/pedrorq/60rtho")
 	)
 	(junction

Commit message: remove per key RGB with LEDs
Replace per-key RGB with 12 underglow LEDs
Removed per-key LEDs U76-U146, RGB1, RGB2 and caps C23-C46
Added LED1-LED12 (SK6812MINI, back side) chained from GPIO19, with caps C17-C22
Parts:
- removed C23, C24, C25, C26, C27, C28, C29, C30, C31, C32, C33, C34, C35, C36, C37, C38, C39, C40, C41, C42, C43, C44, C45, C46: 100n, Capacitor_SMD:C_0603_1608Metric, symbol Device:C
- removed RGB1, RGB2: SK6812MINI-E, Keyboard RGB:RGB_SK6812MINI-E, symbol CherryMX:RGB_(edited)
- removed U100, U101, U102, U103, U104, U105, U106, U107, U108, U109, U110, U111, U112, U113, U114, U115, U116, U117, U118, U119, U120, U121, U122, U123, U124, U125, U126, U127, U128, U129, U130, U131, U132, U133, U134, U135, U136, U137, U138, U139, U140, U141, U142, U143, U144, U145, U146, U76, U77, U78, U79, U80, U81, U82, U83, U84, U85, U86, U87, U88, U89, U90, U91, U92, U93, U94, U95, U96, U97, U98, U99: RGB_(edited), 3rdparty:SK6812-MINI-E, symbol CherryMX:RGB_(edited)
- added LED1, LED10, LED11, LED12, LED2, LED3, LED4, LED5, LED6, LED7, LED8, LED9: SK6812MINI, LED_SMD:LED_SK6812MINI_PLCC4_3.5x3.5mm_P1.75mm, symbol CherryMX:RGB_(edited)
Connections:
- net +3V3: now also LED1.1 (VDD), LED10.1 (VDD), LED11.1 (VDD), LED12.1 (VDD), LED2.1 (VDD), LED3.1 (VDD), LED4.1 (VDD), LED5.1 (VDD), LED6.1 (VDD), LED7.1 (VDD), LED8.1 (VDD), LED9.1 (VDD)
- net GND: now also LED1.3 (VSS), LED10.3 (VSS), LED11.3 (VSS), LED12.3 (VSS), LED2.3 (VSS), LED3.3 (VSS), LED4.3 (VSS), LED5.3 (VSS), LED6.3 (VSS), LED7.3 (VSS), LED8.3 (VSS), LED9.3 (VSS)
- net RGBData1: now also U62.30 (GPIO19), LED1.4 (DIN)
- new net UG_1: LED1.2 (DOUT), LED2.4 (DIN)
- new net UG_10: LED10.2 (DOUT), LED11.4 (DIN)
- new net UG_11: LED11.2 (DOUT), LED12.4 (DIN)
- new net UG_2: LED2.2 (DOUT), LED3.4 (DIN)
- new net UG_3: LED3.2 (DOUT), LED4.4 (DIN)
- new net UG_4: LED4.2 (DOUT), LED5.4 (DIN)
- new net UG_5: LED5.2 (DOUT), LED6.4 (DIN)
- new net UG_6: LED6.2 (DOUT), LED7.4 (DIN)
- new net UG_7: LED7.2 (DOUT), LED8.4 (DIN)
- new net UG_8: LED8.2 (DOUT), LED9.4 (DIN)
- new net UG_9: LED10.4 (DIN), LED9.2 (DOUT)
- no-connect marks 16 -> 15
Other:
- note added: "UNDERGLOW (back of PCB, facing down)"
- company: Pedro Quaresma (TheReflex) -> Pierre Constantineau (JPConstantineau)
- title: 60rtho RP2040 -> PyKey60 RP2040

Commit message: Cleanup
removed excess diodes, placed the remaining oned the back, added stabs.
Parts:
- removed D63, D64, D65, D67, D69, D71, D72, D73: D, Diode_SMD:D_SOD-123, symbol Device:D
- removed SW3, SW4: CherryMX, Keyboard Switches:SW_MX_HotSwap_reinforced, symbol CherryMX:CherryMX
- added ST1, ST2, ST3, ST4, ST5: Stabilizer_2u_MX, Keyboard Stabilizer:Stabilizer_Cherry_MX_2.00u, symbol Keyboard Switches:Stabilizer_2u_MX
- added ST6: Stabilizer_2u_MX, Keyboard Stabilizer:Stabilizer_Cherry_MX_6.25u, symbol Keyboard Switches:Stabilizer_6.25u_MX
Connections:
- net COL10: now also U73.2
- net COL11: now also U74.2
- net COL12: now also U75.2
- net COL13: no longer U75.2
- net COL5: no longer U71.2
- net COL6: now also U71.2
- net COL8: no longer U73.2
- net COL9: no longer U74.2
- net QSPICLK: now also U64.6 (CLK)
- net QSPISD0: now also U64.5 (DI/IO_{0})
- net QSPISD2: now also U64.3 (~{WP}/IO_{2})
- net QSPISD3: now also U64.7 (~{HOLD}/~{RESET}/IO_{3})
- net QSPISS: now also U64.1 (~{CS})
- net ROW1: now also U66.1
- net ROW2: now also U67.1
- net ROW4: now also U69.1
- net ROW5: now also U71.1, U73.1, U74.1, U75.1
- net SQPISD1: now also U64.2 (DO/IO_{1})
Other:
- moved on the sheet: C14, R6, R7, SW2, U64
