File: 60rtho.kicad_pcb (KiCad board)
At the start: 2 copper layers, 285 x 95 mm, 232 parts, among them J1 USB_C_Receptacle_USB2.0, J2 Conn_01x03, J3 Conn_01x04, J4 Conn_01x06, SW1 SW_SPST, SW2 SW_SPDT, SW3 CherryMX, SW4 CherryMX, U1 CherryMX_LTST-A683CEGBW, U10 CherryMX_LTST-A683CEGBW, U11 CherryMX_LTST-A683CEGBW, U12 CherryMX_LTST-A683CEGBW, U13 CherryMX_LTST-A683CEGBW, U14 CherryMX_LTST-A683CEGBW, U15 CherryMX_LTST-A683CEGBW, U16 CherryMX_LTST-A683CEGBW, U17 CherryMX_LTST-A683CEGBW, U18 CherryMX_LTST-A683CEGBW, U19 CherryMX_LTST-A683CEGBW, U2 CherryMX_LTST-A683CEGBW, U20 CherryMX_LTST-A683CEGBW, U21 CherryMX_LTST-A683CEGBW, U22 CherryMX_LTST-A683CEGBW, U23 CherryMX_LTST-A683CEGBW, U24 CherryMX_LTST-A683CEGBW, U25 CherryMX_LTST-A683CEGBW, U26 CherryMX_LTST-A683CEGBW, U27 CherryMX_LTST-A683CEGBW, U28 CherryMX_LTST-A683CEGBW, U29 CherryMX_LTST-A683CEGBW, U3 CherryMX_LTST-A683CEGBW, U30 CherryMX_LTST-A683CEGBW, U31 CherryMX_LTST-A683CEGBW, U32 CherryMX_LTST-A683CEGBW, U33 CherryMX_LTST-A683CEGBW, U34 CherryMX_LTST-A683CEGBW, U35 CherryMX_LTST-A683CEGBW, U36 CherryMX_LTST-A683CEGBW, U37 CherryMX_LTST-A683CEGBW, U38 CherryMX_LTST-A683CEGBW, U39 CherryMX_LTST-A683CEGBW, U4 CherryMX_LTST-A683CEGBW, U40 CherryMX_LTST-A683CEGBW, U41 CherryMX_LTST-A683CEGBW, U42 CherryMX_LTST-A683CEGBW, U43 CherryMX_LTST-A683CEGBW, U44 CherryMX_LTST-A683CEGBW, U45 CherryMX_LTST-A683CEGBW, U46 CherryMX_LTST-A683CEGBW, U47 CherryMX_LTST-A683CEGBW, U48 CherryMX_LTST-A683CEGBW, U49 CherryMX_LTST-A683CEGBW, U5 CherryMX_LTST-A683CEGBW, U50 CherryMX_LTST-A683CEGBW, U51 CherryMX_LTST-A683CEGBW, U52 CherryMX_LTST-A683CEGBW, U53 CherryMX_LTST-A683CEGBW, U54 CherryMX_LTST-A683CEGBW, U55 CherryMX_LTST-A683CEGBW, U56 CherryMX_LTST-A683CEGBW, U57 CherryMX_LTST-A683CEGBW, U58 CherryMX_LTST-A683CEGBW, U59 CherryMX_LTST-A683CEGBW, U6 CherryMX_LTST-A683CEGBW, U60 CherryMX_LTST-A683CEGBW, U61 CherryMX_LTST-A683CEGBW, U62 RP2040, U63 USBLC6-2SC6, U64 W25Q128JVS, U65 AMS1117-3.3, U7 CherryMX_LTST-A683CEGBW, U8 CherryMX_LTST-A683CEGBW, U9 CherryMX_LTST-A683CEGBW, Y1 12MHz

Commit message: adjusted schematics and pcb
adjusted schematics and pcb
71 switches centered within the board ✓
Equal left/right margins ✓
All diodes positioned ✓
MCU and support circuitry intact ✓

The remaining work is routing the traces and verifying overlaps
Parts:
- added D64: D, Diode_SMD:D_SOD-123, F.Cu at (338.0, 82.2)
- added D65: D, Diode_SMD:D_SOD-123, F.Cu at (323.7, 101.2)
- added D66: D, Diode_SMD:D_SOD-123, F.Cu at (299.9, 139.3)
- added D67: D, Diode_SMD:D_SOD-123, F.Cu at (330.8, 139.3)
- added D68: D, Diode_SMD:D_SOD-123, F.Cu at (159.4, 158.4)
- added D69: D, Diode_SMD:D_SOD-123, F.Cu at (192.8, 158.4)
- added D70: D, Diode_SMD:D_SOD-123, F.Cu at (230.8, 158.4)
- added D71: D, Diode_SMD:D_SOD-123, F.Cu at (280.9, 158.4)
- added D72: D, Diode_SMD:D_SOD-123, F.Cu at (299.9, 158.4)
- added D73: D, Diode_SMD:D_SOD-123, F.Cu at (318.9, 158.4)
- added U66: CherryMX_LTST-A683CEGBW, CherryMX_PCB_KailhSocket_LTST-A683CEGBW-Rotated-HS:CherryMX_1.00u_PCB_KailhSocket_LTST-A683CEGBW-Rotated-HS, F.Cu at (333.4, 73.8)
- added U67: CherryMX_LTST-A683CEGBW, CherryMX_PCB_KailhSocket_LTST-A683CEGBW-Rotated-HS:CherryMX_1.50u_PCB_KailhSocket_LTST-A683CEGBW-Rotated-HS, F.Cu at (319.1, 92.9)
- added U68: CherryMX_LTST-A683CEGBW, CherryMX_PCB_KailhSocket_LTST-A683CEGBW-Rotated-HS:CherryMX_1.00u_PCB_KailhSocket_LTST-A683CEGBW-Rotated-HS, F.Cu at (295.3, 131.0)
- added U69: CherryMX_LTST-A683CEGBW, CherryMX_PCB_KailhSocket_StabWireBottom_LTST-A683CEGBW-Rotated-HS:CherryMX_2.25u_PCB_KailhSocket_StabWireBottom_LTST-A6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, F.Cu at (326.2, 131.0)
- added U70: CherryMX_LTST-A683CEGBW, CherryMX_PCB_KailhSocket_StabWireBottom_LTST-A683CEGBW-Rotated-HS:CherryMX_2.25u_PCB_KailhSocket_StabWireBottom_LTST-A6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, F.Cu at (154.8, 150.0)
- added U71: CherryMX_LTST-A683CEGBW, CherryMX_PCB_KailhSocket_LTST-A683CEGBW-Rotated-HS:CherryMX_1.25u_PCB_KailhSocket_LTST-A683CEGBW-Rotated-HS, F.Cu at (188.1, 150.0)
- added U72: CherryMX_LTST-A683CEGBW, CherryMX_PCB_KailhSocket_StabWireBottom_LTST-A683CEGBW-Rotated-HS:CherryMX_2.75u_PCB_KailhSocket_StabWireBottom_LTST-A6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, F.Cu at (226.2, 150.0)
- added U73: CherryMX_LTST-A683CEGBW, CherryMX_PCB_KailhSocket_LTST-A683CEGBW-Rotated-HS:CherryMX_1.00u_PCB_KailhSocket_LTST-A683CEGBW-Rotated-HS, F.Cu at (276.2, 150.0)
- added U74: CherryMX_LTST-A683CEGBW, CherryMX_PCB_KailhSocket_LTST-A683CEGBW-Rotated-HS:CherryMX_1.00u_PCB_KailhSocket_LTST-A683CEGBW-Rotated-HS, F.Cu at (295.3, 150.0)
- added U75: CherryMX_LTST-A683CEGBW, CherryMX_PCB_KailhSocket_LTST-A683CEGBW-Rotated-HS:CherryMX_1.00u_PCB_KailhSocket_LTST-A683CEGBW-Rotated-HS, F.Cu at (314.3, 150.0)
- moved U1 14.3 mm to (85.7, 73.8)
- moved U2 14.3 mm to (104.8, 73.8)
- moved U11 14.3 mm to (276.2, 73.8)
- moved U10 14.3 mm to (257.2, 73.8)
- moved U3 14.3 mm to (123.8, 73.8)
- moved U4 14.3 mm to (142.9, 73.8)
- moved U5 14.3 mm to (161.9, 73.8)
- moved U6 14.3 mm to (181.0, 73.8)
- moved U7 14.3 mm to (200.0, 73.8)
- moved U8 14.3 mm to (219.1, 73.8)
- moved U9 14.3 mm to (238.1, 73.8)
- moved U12 14.3 mm to (295.3, 73.8)
- moved U13 14.3 mm to (314.3, 73.8)
- moved D12 14.3 mm to (300.0, 82.2)
- moved D2 14.3 mm to (109.4, 82.1)
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Routing:
- net RGBEXT: track 0.00 -> 306.0 mm, vias 0 -> 3
- net RGBData2: track 303.4 -> 0.00 mm, vias 2 -> 0
- net +3V3: track 1789.7 -> 2001.0 mm, vias 44 -> 68
- net GND: track 234.8 -> 372.5 mm, vias 97 -> 91
- net Net-(U52-DOUT): track 30.6 -> 2.55 mm, vias 2 -> 1
- net (no net): track 25.9 -> 0.00 mm, vias 2 -> 0
- net Net-(U42-DOUT): track 25.9 -> 2.02 mm, vias 2 -> 1
- net Net-(U58-DOUT): track 18.8 -> 0.00 mm, vias 2 -> 0
- net Net-(U15-DOUT): track 18.7 -> 0.00 mm, vias 2 -> 0
- net Net-(U49-DOUT): track 14.0 -> 0.00 mm, vias 2 -> 1
- net Net-(U19-DOUT): track 13.9 -> 0.00 mm, vias 2 -> 0
- net Net-(U1-DOUT): track 15.1 -> 1.39 mm, vias 2 -> 1
- net ROW2: track 350.8 -> 363.0 mm
- net Net-(D27-A): track 12.1 -> 0.00 mm
- net Net-(U26-DOUT): track 14.0 -> 2.10 mm, vias 2 -> 1
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