File: 60rtho.kicad_pcb (KiCad board)
At the start: 2 copper layers, 285 x 95 mm, 289 parts, among them J1 USB_C_Receptacle_USB2.0, J2 Conn_01x03, SW1 SW_SPST, SW2 SW_SPDT, SW3 CherryMX, SW4 CherryMX, U1 CherryMX_LTST-A683CEGBW, U10 CherryMX_LTST-A683CEGBW, U100 RGB_(edited), U101 RGB_(edited), U102 RGB_(edited), U103 RGB_(edited), U104 RGB_(edited), U105 RGB_(edited), U106 RGB_(edited), U107 RGB_(edited), U108 RGB_(edited), U109 RGB_(edited), U11 CherryMX_LTST-A683CEGBW, U110 RGB_(edited), U111 RGB_(edited), U112 RGB_(edited), U113 RGB_(edited), U114 RGB_(edited), U115 RGB_(edited), U116 RGB_(edited), U117 RGB_(edited), U118 RGB_(edited), U119 RGB_(edited), U12 CherryMX_LTST-A683CEGBW, U120 RGB_(edited), U121 RGB_(edited), U122 RGB_(edited), U123 RGB_(edited), U124 RGB_(edited), U125 RGB_(edited), U126 RGB_(edited), U127 RGB_(edited), U128 RGB_(edited), U129 RGB_(edited), U13 CherryMX_LTST-A683CEGBW, U130 RGB_(edited), U131 RGB_(edited), U132 RGB_(edited), U133 RGB_(edited), U134 RGB_(edited), U135 RGB_(edited), U136 RGB_(edited), U137 RGB_(edited), U138 RGB_(edited), U139 RGB_(edited), U14 CherryMX_LTST-A683CEGBW, U140 RGB_(edited), U141 RGB_(edited), U142 RGB_(edited), U143 RGB_(edited), U144 RGB_(edited), U145 RGB_(edited), U146 RGB_(edited), U15 CherryMX_LTST-A683CEGBW, U16 CherryMX_LTST-A683CEGBW, U17 CherryMX_LTST-A683CEGBW, U18 CherryMX_LTST-A683CEGBW, U19 CherryMX_LTST-A683CEGBW, U2 CherryMX_LTST-A683CEGBW, U20 CherryMX_LTST-A683CEGBW, U21 CherryMX_LTST-A683CEGBW, U22 CherryMX_LTST-A683CEGBW, U23 CherryMX_LTST-A683CEGBW, U24 CherryMX_LTST-A683CEGBW, U25 CherryMX_LTST-A683CEGBW, U26 CherryMX_LTST-A683CEGBW, U27 CherryMX_LTST-A683CEGBW, U28 CherryMX_LTST-A683CEGBW, U29 CherryMX_LTST-A683CEGBW, U3 CherryMX_LTST-A683CEGBW, U30 CherryMX_LTST-A683CEGBW, U31 CherryMX_LTST-A683CEGBW, U32 CherryMX_LTST-A683CEGBW, U33 CherryMX_LTST-A683CEGBW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

Commit message: Place LEDs U76-U146 above their switches
Each LED placed 5.08mm above its switch, rotated 90° to match RGB1/RGB2.
Removed KiCad lock files and added .gitignore for *.lck and .history.
Parts:
- moved U87 232.6 mm to (295.3, 68.7), turned to 90 degrees
- moved U86 217.8 mm to (276.2, 68.7), turned to 90 degrees
- moved U89 214.0 mm to (323.9, 68.7), turned to 90 degrees
- moved U88 204.0 mm to (314.3, 68.7), turned to 90 degrees
- moved U85 203.8 mm to (257.2, 68.7), turned to 90 degrees
- moved U129 200.9 mm to (333.4, 87.8), turned to 90 degrees
- moved U138 198.8 mm to (333.4, 68.7), turned to 90 degrees
- moved U123 191.5 mm to (276.2, 87.8), turned to 90 degrees
- moved U84 190.7 mm to (238.1, 68.7), turned to 90 degrees
- moved U130 185.8 mm to (326.2, 106.8), turned to 90 degrees
- moved U128 184.3 mm to (314.3, 87.8), turned to 90 degrees
- moved U83 178.9 mm to (219.1, 68.7), turned to 90 degrees
- moved U122 178.5 mm to (257.2, 87.8), turned to 90 degrees
- moved U139 178.4 mm to (319.1, 87.8), turned to 90 degrees
- moved U132 175.7 mm to (335.8, 144.9), turned to 90 degrees
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Routing:
- net (no net): track 711.5 -> 704.1 mm, vias 69 -> 66
- net GND: track 347.8 -> 353.8 mm, vias 90 -> 92
- net RGBData1: track 0.00 -> 1.39 mm, vias 0 -> 1

Commit message: remove per key RGB with LEDs
Replace per-key RGB with 12 underglow LEDs
Removed per-key LEDs U76-U146, RGB1, RGB2 and caps C23-C46
Added LED1-LED12 (SK6812MINI, back side) chained from GPIO19, with caps C17-C22
Parts:
- removed C23, C24, C25, C26, C27, C28, C29, C30, C31, C32, C33, C34, C35, C36, C37, C38, C39, C40, C41, C42, C43, C44, C45, C46: 100n, Capacitor_SMD:C_0603_1608Metric
- removed RGB1, RGB2: SK6812MINI-E, Keyboard RGB:RGB_SK6812MINI-E
- removed U100, U101, U102, U103, U104, U105, U106, U107, U108, U109, U110, U111, U112, U113, U114, U115, U116, U117, U118, U119, U120, U121, U122, U123, U124, U125, U126, U127, U128, U129, U130, U131, U132, U133, U134, U135, U136, U137, U138, U139, U140, U141, U142, U143, U144, U145, U146, U76, U77, U78, U79, U80, U81, U82, U83, U84, U85, U86, U87, U88, U89, U90, U91, U92, U93, U94, U95, U96, U97, U98, U99: RGB_(edited), 3rdparty:SK6812-MINI-E
- added LED1: SK6812MINI, LED_SMD:LED_SK6812MINI_PLCC4_3.5x3.5mm_P1.75mm, B.Cu at (144.8, 155.5)
- added LED10: SK6812MINI, LED_SMD:LED_SK6812MINI_PLCC4_3.5x3.5mm_P1.75mm, B.Cu at (325.8, 150.2)
- added LED11: SK6812MINI, LED_SMD:LED_SK6812MINI_PLCC4_3.5x3.5mm_P1.75mm, B.Cu at (259.5, 146.8)
- added LED12: SK6812MINI, LED_SMD:LED_SK6812MINI_PLCC4_3.5x3.5mm_P1.75mm, B.Cu at (207.5, 155.5)
- added LED2: SK6812MINI, LED_SMD:LED_SK6812MINI_PLCC4_3.5x3.5mm_P1.75mm, B.Cu at (89.0, 151.0)
- added LED3: SK6812MINI, LED_SMD:LED_SK6812MINI_PLCC4_3.5x3.5mm_P1.75mm, B.Cu at (65.8, 111.5)
- added LED4: SK6812MINI, LED_SMD:LED_SK6812MINI_PLCC4_3.5x3.5mm_P1.75mm, B.Cu at (90.8, 68.2)
- added LED5: SK6812MINI, LED_SMD:LED_SK6812MINI_PLCC4_3.5x3.5mm_P1.75mm, B.Cu at (147.8, 68.2)
- added LED6: SK6812MINI, LED_SMD:LED_SK6812MINI_PLCC4_3.5x3.5mm_P1.75mm, B.Cu at (204.8, 68.2)
- added LED7: SK6812MINI, LED_SMD:LED_SK6812MINI_PLCC4_3.5x3.5mm_P1.75mm, B.Cu at (261.8, 68.2)
- added LED8: SK6812MINI, LED_SMD:LED_SK6812MINI_PLCC4_3.5x3.5mm_P1.75mm, B.Cu at (310.2, 68.2)
- added LED9: SK6812MINI, LED_SMD:LED_SK6812MINI_PLCC4_3.5x3.5mm_P1.75mm, B.Cu at (343.8, 111.5)
- moved C21 236.0 mm to (343.8, 115.5)
- moved C20 205.1 mm to (266.1, 68.2), turned to 90 degrees
- moved C19 151.9 mm to (152.1, 68.2), turned to 90 degrees
- moved C18 61.3 mm to (65.8, 115.5)
- moved C22 32.3 mm to (259.5, 142.8)
- moved C17 20.8 mm to (144.8, 151.5)
Connections:
- D63 pad 1: Net-(D63-K) -> unconnected-(D63-K-Pad1)
- SW4 pad 2: Net-(U130-DIN) -> unconnected-(SW4-~-Pad2)
- U62 pad 30: unconnected-(U62-GPIO19-Pad30) -> RGBData1
Routing:
- net (no net): track 704.1 -> 1771.3 mm, vias 66 -> 73
- net RGBEXT: track 306.0 -> 0.00 mm, vias 3 -> 0
- net RGBData3: track 289.2 -> 0.00 mm, vias 2 -> 0
- net RGBData4: track 284.1 -> 0.00 mm, vias 2 -> 0
- net RGBData5: track 282.0 -> 0.00 mm, vias 2 -> 0
- net +3V3: track 2001.0 -> 2067.3 mm, vias 68 -> 70
- net GND: track 353.8 -> 381.7 mm
