File: 60rtho.kicad_pcb (KiCad board)
At the start: 2 copper layers, 285 x 95 mm, 204 parts, among them J1 USB_C_Receptacle_USB2.0, J2 Conn_01x03, SW1 SW_SPST, SW2 SW_SPDT, SW3 CherryMX, SW4 CherryMX, U1 CherryMX_LTST-A683CEGBW, U10 CherryMX_LTST-A683CEGBW, U11 CherryMX_LTST-A683CEGBW, U12 CherryMX_LTST-A683CEGBW, U13 CherryMX_LTST-A683CEGBW, U14 CherryMX_LTST-A683CEGBW, U15 CherryMX_LTST-A683CEGBW, U16 CherryMX_LTST-A683CEGBW, U17 CherryMX_LTST-A683CEGBW, U18 CherryMX_LTST-A683CEGBW, U19 CherryMX_LTST-A683CEGBW, U2 CherryMX_LTST-A683CEGBW, U20 CherryMX_LTST-A683CEGBW, U21 CherryMX_LTST-A683CEGBW, U22 CherryMX_LTST-A683CEGBW, U23 CherryMX_LTST-A683CEGBW, U24 CherryMX_LTST-A683CEGBW, U25 CherryMX_LTST-A683CEGBW, U26 CherryMX_LTST-A683CEGBW, U27 CherryMX_LTST-A683CEGBW, U28 CherryMX_LTST-A683CEGBW, U29 CherryMX_LTST-A683CEGBW, U3 CherryMX_LTST-A683CEGBW, U30 CherryMX_LTST-A683CEGBW, U31 CherryMX_LTST-A683CEGBW, U32 CherryMX_LTST-A683CEGBW, U33 CherryMX_LTST-A683CEGBW, U34 CherryMX_LTST-A683CEGBW, U35 CherryMX_LTST-A683CEGBW, U36 CherryMX_LTST-A683CEGBW, U37 CherryMX_LTST-A683CEGBW, U38 CherryMX_LTST-A683CEGBW, U39 CherryMX_LTST-A683CEGBW, U4 CherryMX_LTST-A683CEGBW, U40 CherryMX_LTST-A683CEGBW, U41 CherryMX_LTST-A683CEGBW, U42 CherryMX_LTST-A683CEGBW, U43 CherryMX_LTST-A683CEGBW, U44 CherryMX_LTST-A683CEGBW, U45 CherryMX_LTST-A683CEGBW, U46 CherryMX_LTST-A683CEGBW, U47 CherryMX_LTST-A683CEGBW, U48 CherryMX_LTST-A683CEGBW, U49 CherryMX_LTST-A683CEGBW, U5 CherryMX_LTST-A683CEGBW, U50 CherryMX_LTST-A683CEGBW, U51 CherryMX_LTST-A683CEGBW, U52 CherryMX_LTST-A683CEGBW, U53 CherryMX_LTST-A683CEGBW, U54 CherryMX_LTST-A683CEGBW, U55 CherryMX_LTST-A683CEGBW, U56 CherryMX_LTST-A683CEGBW, U57 CherryMX_LTST-A683CEGBW, U58 CherryMX_LTST-A683CEGBW, U59 CherryMX_LTST-A683CEGBW, U6 CherryMX_LTST-A683CEGBW, U60 CherryMX_LTST-A683CEGBW, U61 CherryMX_LTST-A683CEGBW, U62 RP2040, U63 USBLC6-2SC6, U64 W25Q128JVS, U65 AMS1117-3.3, U66 CherryMX_LTST-A683CEGBW, U67 CherryMX_LTST-A683CEGBW, U68 CherryMX_LTST-A683CEGBW, U69 CherryMX_LTST-A683CEGBW, U7 CherryMX_LTST-A683CEGBW, U70 CherryMX_LTST-A683CEGBW, U71 CherryMX_LTST-A683CEGBW, U72 CherryMX_LTST-A683CEGBW, U73 CherryMX_LTST-A683CEGBW, U74 CherryMX_LTST-A683CEGBW, U75 CherryMX_LTST-A683CEGBW, U8 CherryMX_LTST-A683CEGBW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

Commit message: Cleanup
removed excess diodes, placed the remaining oned the back, added stabs.
Parts:
- removed D63, D65, D67, D69, D71, D72, D73: D, Diode_SMD:D_SOD-123
- removed SW3, SW4: CherryMX, Keyboard Switches:SW_MX_HotSwap_reinforced
- added ST1: Stabilizer_2u_MX, Keyboard Stabilizer:Stabilizer_Cherry_MX_2.00u, F.Cu at (323.9, 73.8)
- added ST2: Stabilizer_2u_MX, Keyboard Stabilizer:Stabilizer_Cherry_MX_2.00u, F.Cu at (326.2, 111.9)
- added ST3: Stabilizer_2u_MX, Keyboard Stabilizer:Stabilizer_Cherry_MX_2.00u, F.Cu at (326.2, 131.0)
- added ST4: Stabilizer_2u_MX, Keyboard Stabilizer:Stabilizer_Cherry_MX_2.00u, F.Cu at (226.2, 150.0)
- added ST5: Stabilizer_2u_MX, Keyboard Stabilizer:Stabilizer_Cherry_MX_2.00u, F.Cu at (154.8, 150.0)
- added ST6: Stabilizer_2u_MX, Keyboard Stabilizer:Stabilizer_Cherry_MX_6.25u, F.Cu at (192.9, 150.0)
- D64, D66, D68, D70: moved to B.Cu
- moved H7 107.9 mm to (69.9, 79.3)
- moved D61 20.0 mm to (343.2, 146.7)
- moved D53 15.4 mm to (335.7, 129.3)
- moved LED11 11.8 mm to (252.6, 156.3)
- moved D60 10.6 mm to (323.4, 144.8)
- moved D66 10.4 mm to (303.2, 129.5), turned to -90 degrees
- moved D54 7.74 mm to (82.8, 148.1)
- moved LED1 7.55 mm to (137.2, 156.1)
- moved LED10 5.87 mm to (323.9, 155.8)
- moved LED2 5.40 mm to (85.8, 155.4)
- moved LED8 4.59 mm to (305.7, 67.8)
- moved D64 4.11 mm to (336.0, 85.8), turned to 180 degrees
- moved D70 3.79 mm to (232.2, 154.8), turned to 180 degrees
- moved LED12 0.96 mm to (208.5, 155.5)
- turned D68 to 180 degrees
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Connections:
- U64 pad 1: unconnected-(U64-~{CS}-Pad1) -> /QSPISS
- U64 pad 2: unconnected-(U64-DO/IO_{1}-Pad2) -> /SQPISD1
- U64 pad 3: unconnected-(U64-~{WP}/IO_{2}-Pad3) -> /QSPISD2
- U64 pad 5: unconnected-(U64-DI/IO_{0}-Pad5) -> /QSPISD0
- U64 pad 6: unconnected-(U64-CLK-Pad6) -> /QSPICLK
- U64 pad 7: unconnected-(U64-~{HOLD}/~{RESET}/IO_{3}-Pad7) -> /QSPISD3
- U67 pad 1: Net-(D65-A) -> ROW2
- U69 pad 1: Net-(D67-A) -> ROW4
- U71 pad 1: Net-(D69-A) -> ROW5
- U71 pad 2: COL5 -> COL6
- U73 pad 1: Net-(D71-A) -> ROW5
- U73 pad 2: COL8 -> COL10
- U74 pad 1: Net-(D72-A) -> ROW5
- U74 pad 2: COL9 -> COL11
- U75 pad 1: Net-(D73-A) -> ROW5
- U75 pad 2: COL13 -> COL12
Routing:
- net (no net): track 1771.3 -> 0.00 mm, vias 73 -> 1
- net +3V3: track 2067.3 -> 599.4 mm, vias 70 -> 7
- net ROW1: track 386.3 -> 0.00 mm, vias 16 -> 0
- net ROW4: track 302.8 -> 0.00 mm, vias 14 -> 0
- net COL13: track 196.7 -> 0.00 mm, vias 2 -> 0
- net unconnected-(U62-GPIO29_ADC3-Pad41): track 176.9 -> 0.00 mm, vias 2 -> 0
- net ROW2: track 363.0 -> 236.7 mm, vias 16 -> 4
- net LED: track 119.7 -> 0.00 mm, vias 4 -> 0
- net Data-: track 114.0 -> 0.00 mm
- net Data+: track 112.8 -> 0.00 mm
- net COL2: track 171.6 -> 89.5 mm, vias 3 -> 2
- net GND: track 381.7 -> 312.6 mm, vias 92 -> 78
- net COL8: track 149.3 -> 84.1 mm, vias 5 -> 2
- net COL10: track 182.0 -> 116.9 mm
- net unconnected-(U62-GPIO28_ADC2-Pad40): track 55.8 -> 0.00 mm, vias 1 -> 0
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Other:
- board text removed: "GND 3V3 SCK TX RX CS"
- board text removed: "GND 3V3 SDA SCL"
- board text removed: "I2C1"
- board text removed: "SPI1"
- board text removed: "TheReflex 2026"

Commit message: Draft matrix + underglow routing (Freerouting)
   Routed rows, columns, diode links and underglow chain only. MCU end left unconnected.
   Removed old PyKey60 traces for those nets (371 segments, 43 vias).
   Rows/links on B.Cu, columns on F.Cu. 80/95 nets complete, 21 vias, no clearance violations.
   29 connections still open (mostly bottom row and columns between home and shift rows).
Routing:
- net ROW4: track 0.00 -> 386.6 mm
- net COL8: track 84.1 -> 366.0 mm, vias 2 -> 0
- net ROW1: track 0.00 -> 271.7 mm
- net ROW5: track 206.8 -> 31.7 mm
- net ROW3: track 361.8 -> 217.4 mm, vias 15 -> 0
- net COL13: track 0.00 -> 133.1 mm
- net COL12: track 173.5 -> 65.1 mm, vias 2 -> 0
- net COL14: track 193.3 -> 93.4 mm, vias 2 -> 0
- net COL9: track 98.4 -> 19.7 mm, vias 2 -> 0
- net /UG_8: track 0.00 -> 76.8 mm, vias 0 -> 1
- net /UG_10: track 0.00 -> 76.3 mm, vias 0 -> 2
- net COL6: track 65.2 -> 136.2 mm
- net /UG_2: track 0.00 -> 62.8 mm, vias 0 -> 2
- net COL1: track 143.4 -> 82.1 mm, vias 2 -> 0
- net /UG_3: track 0.00 -> 59.3 mm, vias 0 -> 2
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